Commit message: Cleaning

File: simulation/urdf/quadrotor.gazebo.xacro (robot description, xacro)
@@ -3,9 +3,4 @@
     <xacro:include filename="$(find m100_simulation)/simulation/urdf/quadrotor.urdf.xacro" />
     <xacro:include filename="$(find hector_quadrotor_gazebo)/urdf/quadrotor_plugins.gazebo.xacro" />
-    <!-- Real Sense -->
-    <!-- <xacro:include filename="$(find realsense2_description)/urdf/_d435.urdf.xacro" />
-    <xacro:sensor_d435 name="camera" topics_ns="camera" parent="base_link" publish_pointcloud="true">
-        <origin xyz="0.05 0 -0.05" rpy="0 0 0" />
-    </xacro:sensor_d435>  -->
     <!-- Ouster -->
     <xacro:include filename="$(find ouster_os1_64)/urdf/os1_64.urdf.xacro"/>
@@ -15,14 +10,3 @@
         <origin xyz="0.0 0 0.14" rpy="0 0 0"/>
     </xacro:os1_64>
-    <!-- Livox MID360 -->
-    <!-- <xacro:include filename="$(find ouster_os1_64)/urdf/os1_64.urdf.xacro"/>
-    <xacro:os1_64 parent="base_link" name="ouster" prefix="os1_cloud_node" hz="10" samples="256" gpu="true"
-            reduced="false" min_range="0.09" min_angle_v="-7" max_angle_v="52"> -->
-        <!-- 15 deg -->
-        <!-- <origin xyz="0.0 0 0.14" rpy="0  0.2617993878 0" />  -->
-        <!-- 20 deg -->
-        <!-- <origin xyz="0.0 0 0.14" rpy="0 0.3490658504 0" />  -->
-        <!-- 30 deg -->
-        <!-- <origin xyz="0.0 0 0.14" rpy="0 0.5235987756 0" />  -->
-    <!-- </xacro:os1_64> -->
 </robot>

File: simulation/urdf/quadrotor_base.urdf.xacro (robot description, xacro)
@@ -17,5 +17,4 @@
         </geometry>
       </visual>
-      <!-- REDUCED -->
       <collision>
         <origin xyz="0 0 0" rpy="0 0 0" />
@@ -24,29 +23,4 @@
         </geometry>
       </collision>
-      <!-- REALISTIC -->
-      <!-- <collision>
-        <origin xyz="0.235 0.235 0" rpy="0 0 0" />
-        <geometry>
-          <cylinder radius="0.17" length="0.23"/>
-        </geometry>
-      </collision>
-      <collision>
-      <origin xyz="0.235 -0.235 0" rpy="0 0 0" />
-        <geometry>
-          <cylinder radius="0.17" length="0.23"/>
-        </geometry>
-      </collision>
-      <collision>
-      <origin xyz="-0.235 0.235 0" rpy="0 0 0" />
-        <geometry>
-          <cylinder radius="0.17" length="0.23"/>
-        </geometry>
-      </collision>
-      <collision>
-      <origin xyz="-0.235 -0.235 0" rpy="0 0 0" />
-        <geometry>
-          <cylinder radius="0.17" length="0.23"/>
-        </geometry>
-      </collision> -->
     </link>
     <gazebo reference="base_link">
@@ -81,27 +55,4 @@
       </sensor>
     </gazebo>
-    <!-- <gazebo reference="base_link">
-      <sensor type="ray" name="LidarLite">
-          <pose>0.03 -0.15 0.13 0 -1.57 0</pose>
-          <visualize>true</visualize>
-          <update_rate>50</update_rate>
-          <ray>
-            <range>
-                <min>0.05</min>
-                <max>150</max>
-                <resolution>0.02</resolution>
-            </range>
-          </ray>
-          <plugin filename="libgazebo_ros_range.so" name="gazebo_ros_range">
-            <gaussianNoise>0.0</gaussianNoise>
-            <alwaysOn>true</alwaysOn>
-            <updateRate>50</updateRate>
-            <topicName>ceiling/lidarlite3/range</topicName>
-            <frameName>ceiling/lidarlite3</frameName>
-            <radiation>INFRARED</radiation>
-            <fov>0</fov>
-          </plugin>
-      </sensor>
-    </gazebo> -->
     <gazebo reference="base_link">
       <sensor type="ray" name="LidarLite">
@@ -137,12 +88,7 @@
             <frameName>ceiling/lidarlite3</frameName>
             <radiation>INFRARED</radiation>
-            <!-- <fov>0</fov> -->
           </plugin>
       </sensor>
     </gazebo>
-    <!-- Sonar height sensor -->
-    <!-- <xacro:sonar_sensor name="sonar" parent="base_link" ros_topic="sonar_height" update_rate="10" min_range="0.03" max_range="3.0" field_of_view="${40*pi/180}" ray_count="3">
-      <origin xyz="-0.16 0.0 -0.012" rpy="0 ${90*pi/180} 0"/>
-    </xacro:sonar_sensor> -->
   </xacro:macro>
 </robot>
